File: hardware/Led_Controller.sch (KiCad schematic (older format))
At the start: 15 parts, among them U5 IS31FL3733

Commit message: Update Led_Controller.sch
Parts:
- C19, C20, C21, C22, C23, C24, C25: footprint Capacitors_SMD:C_0603_HandSoldering -> Capacitor_SMD:C_0603_1608Metric_Pad1.05x0.95mm_HandSolder
- C7: footprint Capacitors_SMD:C_1206_HandSoldering -> Capacitor_SMD:C_1206_3216Metric_Pad1.42x1.75mm_HandSolder
- R4, R5, R6, R7, R8, R9: footprint Resistors_SMD:R_0603_HandSoldering -> Resistor_SMD:R_0603_1608Metric_Pad1.05x0.95mm_HandSolder
- U5: footprint Housings_DFN_QFN:UQFN-48-1EP_6x6mm_Pitch0.4mm -> Package_DFN_QFN:UQFN-48-1EP_6x6mm_P0.4mm_EP4.45x4.45mm
Changed lines of the file:
@@
 F 0 "U5" H 9650 4600 60  0000 C CNN
 F 1 "IS31FL3733" H 9200 6150 60  0000 C CNN
-F 2 "Housings_DFN_QFN:UQFN-48-1EP_6x6mm_Pitch0.4mm" H 9650 4600 60  0001 C CNN
+F 2 "Package_DFN_QFN:UQFN-48-1EP_6x6mm_P0.4mm_EP4.45x4.45mm" H 9650 4600 60  0001 C CNN
 F 3 "" H 9650 4600 60  0001 C CNN
 	1    9100 4850
@@
 F 0 "R4" V 7930 6400 50  0000 C CNN
 F 1 "100k" V 7850 6400 50  0000 C CNN
-F 2 "Resistors_SMD:R_0603_HandSoldering" V 7780 6400 50  0001 C CNN
+F 2 "Resistor_SMD:R_0603_1608Metric_Pad1.05x0.95mm_HandSolder" V 7780 6400 50  0001 C CNN
 F 3 "" H 7850 6400 50  0000 C CNN
 	1    7850 6400
@@
 F 0 "R7" V 7780 6300 50  0000 C CNN
 F 1 "100k" V 7700 6300 50  0000 C CNN
-F 2 "Resistors_SMD:R_0603_HandSoldering" V 7630 6300 50  0001 C CNN
+F 2 "Resistor_SMD:R_0603_1608Metric_Pad1.05x0.95mm_HandSolder" V 7630 6300 50  0001 C CNN
 F 3 "" H 7700 6300 50  0000 C CNN
 	1    7700 6300
@@
 F 0 "R5" V 7780 5600 50  0000 C CNN
 F 1 "100k" V 7700 5600 50  0000 C CNN
-F 2 "Resistors_SMD:R_0603_HandSoldering" V 7630 5600 50  0001 C CNN
+F 2 "Resistor_SMD:R_0603_1608Metric_Pad1.05x0.95mm_HandSolder" V 7630 5600 50  0001 C CNN
 F 3 "" H 7700 5600 50  0000 C CNN
 	1    7700 5600
@@
 F 0 "R8" V 7930 5600 50  0000 C CNN
 F 1 "1k" V 7850 5600 50  0000 C CNN
-F 2 "Resistors_SMD:R_0603_HandSoldering" V 7780 5600 50  0001 C CNN
+F 2 "Resistor_SMD:R_0603_1608Metric_Pad1.05x0.95mm_HandSolder" V 7780 5600 50  0001 C CNN
 F 3 "" H 7850 5600 50  0000 C CNN
 	1    7850 5600
@@
 F 0 "R9" V 8080 5600 50  0000 C CNN
 F 1 "1k" V 8000 5600 50  0000 C CNN
-F 2 "Resistors_SMD:R_0603_HandSoldering" V 7930 5600 50  0001 C CNN
+F 2 "Resistor_SMD:R_0603_1608Metric_Pad1.05x0.95mm_HandSolder" V 7930 5600 50  0001 C CNN
 F 3 "" H 8000 5600 50  0000 C CNN
 	1    8000 5600
@@
 F 0 "C19" H 7175 3750 50  0000 L CNN
 F 1 "470nF" H 7175 3550 50  0000 L CNN
-F 2 "Capacitors_SMD:C_0603_HandSoldering" H 7188 3500 50  0001 C CNN
+F 2 "Capacitor_SMD:C_0603_1608Metric_Pad1.05x0.95mm_HandSolder" H 7188 3500 50  0001 C CNN
 F 3 "" H 7150 3650 50  0000 C CNN
 	1    7150 3650
@@
 F 0 "C20" H 6925 3750 50  0000 L CNN
 F 1 "100nF" H 6925 3550 50  0000 L CNN
-F 2 "Capacitors_SMD:C_0603_HandSoldering" H 6938 3500 50  0001 C CNN
+F 2 "Capacitor_SMD:C_0603_1608Metric_Pad1.05x0.95mm_HandSolder" H 6938 3500 50  0001 C CNN
 F 3 "" H 6900 3650 50  0000 C CNN
 	1    6900 3650
@@
 	10400 7350 10150 7350
 Wire Wire Line
-	10400 7050 10400 7450
+	10400 7050 10400 7150
 Connection ~ 10400 7150
 Connection ~ 10400 7350
@@
 	8250 7100 8000 7100
 Wire Wire Line
-	8000 6850 8000 7750
-Wire Wire Line
-	8000 6850 8250 6850
+	8000 6850 8000 7100
+Wire Wire Line
+	8000 6850 8150 6850
 Connection ~ 8000 7100
 Wire Wire Line
@@
 	7850 6550 7850 6600
 Wire Wire Line
-	7500 6150 8250 6150
-Wire Wire Line
-	7500 6050 8250 6050
-Wire Wire Line
-	7500 5950 8250 5950
-Wire Wire Line
-	7500 5850 8250 5850
+	7500 6150 7700 6150
+Wire Wire Line
+	7500 6050 7700 6050
+Wire Wire Line
+	7500 5950 7850 5950
+Wire Wire Line
+	7500 5850 8000 5850
 Wire Wire Line
 	7700 6450 7700 6600
@@
 Connection ~ 8000 5850
 Wire Wire Line
-	7700 5250 7700 5450
+	7700 5250 7700 5350
 Wire Wire Line
 	7850 5450 7850 5350
@@
 	8000 5350 8000 5450
 Wire Wire Line
-	7700 5350 8000 5350
+	7700 5350 7850 5350
 Connection ~ 7700 5350
 Connection ~ 7850 5350
@@
 	10150 6250 10450 6250
 Wire Wire Line
-	6900 3500 8250 3500
+	6900 3500 7150 3500
 Wire Wire Line
 	6900 3500 6900 3350
 Connection ~ 6900 3500
 Wire Wire Line
-	6900 3800 6900 4400
-Wire Wire Line
-	7400 3700 8250 3700
+	6900 3800 6900 4000
+Wire Wire Line
+	7400 3700 7600 3700
 Connection ~ 7150 3500
 $Comp
@@
 F 0 "C22" H 7625 3950 50  0000 L CNN
 F 1 "470nF" H 7625 3750 50  0000 L CNN
-F 2 "Capacitors_SMD:C_0603_HandSoldering" H 7638 3700 50  0001 C CNN
+F 2 "Capacitor_SMD:C_0603_1608Metric_Pad1.05x0.95mm_HandSolder" H 7638 3700 50  0001 C CNN
 F 3 "" H 7600 3850 50  0000 C CNN
 	1    7600 3850
@@
 F 0 "C21" H 7425 3950 50  0000 L CNN
 F 1 "100nF" H 7425 3750 50  0000 L CNN
-F 2 "Capacitors_SMD:C_0603_HandSoldering" H 7438 3700 50  0001 C CNN
+F 2 "Capacitor_SMD:C_0603_1608Metric_Pad1.05x0.95mm_HandSolder" H 7438 3700 50  0001 C CNN
 F 3 "" H 7400 3850 50  0000 C CNN
 	1    7400 3850
@@
 Connection ~ 7600 3700
 Wire Wire Line
-	6900 4000 7600 4000
+	6900 4000 7400 4000
 Connection ~ 6900 4000
 Connection ~ 7400 4000
@@
 	8250 3850 8000 3850
 Wire Wire Line
-	8000 3500 8000 3950
-Wire Wire Line
-	7850 3950 8250 3950
+	8000 3500 8000 3850
+Wire Wire Line
+	7850 3950 8000 3950
 $Comp
 L Device:C C24
@@
 F 0 "C24" H 8025 4200 50  0000 L CNN
 F 1 "470nF" H 8025 4000 50  0000 L CNN
-F 2 "Capacitors_SMD:C_0603_HandSoldering" H 8038 3950 50  0001 C CNN
+F 2 "Capacitor_SMD:C_0603_1608Metric_Pad1.05x0.95mm_HandSolder" H 8038 3950 50  0001 C CNN
 F 3 "" H 8000 4100 50  0000 C CNN
 	1    8000 4100
@@
 F 0 "C23" H 7875 4200 50  0000 L CNN
 F 1 "100nF" H 7875 4000 50  0000 L CNN
-F 2 "Capacitors_SMD:C_0603_HandSoldering" H 7888 3950 50  0001 C CNN
+F 2 "Capacitor_SMD:C_0603_1608Metric_Pad1.05x0.95mm_HandSolder" H 7888 3950 50  0001 C CNN
 F 3 "" H 7850 4100 50  0000 C CNN
 	1    7850 4100
@@
 $EndComp
 Wire Wire Line
-	6900 4250 8000 4250
+	6900 4250 7850 4250
 Connection ~ 6900 4250
 Connection ~ 7850 4250
@@
 F 0 "C25" H 11425 3800 50  0000 L CNN
 F 1 "470nF" H 11425 3600 50  0000 L CNN
-F 2 "Capacitors_SMD:C_0603_HandSoldering" H 11438 3550 50  0001 C CNN
+F 2 "Capacitor_SMD:C_0603_1608Metric_Pad1.05x0.95mm_HandSolder" H 11438 3550 50  0001 C CNN
 F 3 "" H 11400 3700 50  0000 C CNN
 	1    11400 3700
@@
 Connection ~ 8000 7450
 Wire Wire Line
-	11400 3400 11400 3550
+	11400 3400 11400 3500
 Connection ~ 11400 3500
 Wire Wire Line
@@
 F 0 "C7" H 5625 3350 50  0000 L CNN
 F 1 "22uF" H 5625 3150 50  0000 L CNN
-F 2 "Capacitors_SMD:C_1206_HandSoldering" H 5638 3100 50  0001 C CNN
+F 2 "Capacitor_SMD:C_1206_3216Metric_Pad1.42x1.75mm_HandSolder" H 5638 3100 50  0001 C CNN
 F 3 "" H 5600 3250 50  0000 C CNN
 	1    5600 3250
@@
 F 0 "R6" V 6630 7250 50  0000 C CNN
 F 1 "20k" V 6550 7250 50  0000 C CNN
-F 2 "Resistors_SMD:R_0603_HandSoldering" V 6480 7250 50  0001 C CNN
+F 2 "Resistor_SMD:R_0603_1608Metric_Pad1.05x0.95mm_HandSolder" V 6480 7250 50  0001 C CNN
 F 3 "" H 6550 7250 50  0000 C CNN
 	1    6550 7250
@@
 NoConn ~ 10150 6050
 NoConn ~ 10150 6150
+Wire Wire Line
+	10400 7150 10400 7350
+Wire Wire Line
+	10400 7350 10400 7450
+Wire Wire Line
+	8000 7100 8000 7450
+Wire Wire Line
+	8150 6850 8250 6850
+Wire Wire Line
+	7700 6150 8250 6150
+Wire Wire Line
+	7700 6050 8250 6050
+Wire Wire Line
+	7850 5950 8250 5950
+Wire Wire Line
+	8000 5850 8250 5850
+Wire Wire Line
+	7700 5350 7700 5450
+Wire Wire Line
+	7850 5350 8000 5350
+Wire Wire Line
+	7150 3500 7600 3500
+Wire Wire Line
+	7600 3700 8250 3700
+Wire Wire Line
+	6900 4000 6900 4250
+Wire Wire Line
+	7400 4000 7600 4000
+Wire Wire Line
+	8000 3950 8250 3950
+Wire Wire Line
+	6900 4250 6900 4400
+Wire Wire Line
+	7850 4250 8000 4250
+Wire Wire Line
+	7600 3500 8000 3500
+Wire Wire Line
+	8000 3500 8250 3500
+Wire Wire Line
+	8000 3850 8000 3950
+Wire Wire Line
+	8000 7450 8000 7750
+Wire Wire Line
+	11400 3500 11400 3550
 $EndSCHEMATC
