File: hardware/TCKB.sch (KiCad schematic (older format))
At the start: 20 parts, among them J1 USB-MB-H, P2 CONN_01X04, U1 STM32F042C6Tx, U3 MCP1700T-3002E/TT, Y1 Crystal

Commit message: Update TCKB.sch
Parts:
- C1, C10, C11, C2, C3, C4, C5, C6, C8, C9: footprint Capacitors_SMD:C_0603_HandSoldering -> Capacitor_SMD:C_0603_1608Metric_Pad1.05x0.95mm_HandSolder
- DBG1: footprint Pin_Headers:Pin_Header_Straight_1x08_Pitch2.54mm -> Connector_PinHeader_2.54mm:PinHeader_1x08_P2.54mm_Vertical
- EXT1: footprint Pin_Headers:Pin_Header_Straight_1x06_Pitch2.54mm -> Connector_PinHeader_2.54mm:PinHeader_1x06_P2.54mm_Vertical
- P2: footprint Pin_Headers:Pin_Header_Straight_1x04_Pitch2.54mm -> Connector_PinHeader_2.54mm:PinHeader_1x04_P2.54mm_Vertical
- R1, R2, R3: footprint Resistors_SMD:R_0603_HandSoldering -> Resistor_SMD:R_0603_1608Metric_Pad1.05x0.95mm_HandSolder
- U1: footprint Housings_QFP:LQFP-48_7x7mm_Pitch0.5mm -> Package_QFP:LQFP-48_7x7mm_P0.5mm
- U3: footprint TO_SOT_Packages_SMD:SOT-23 -> Package_TO_SOT_SMD:SOT-23
- Y1: footprint Crystals:ABM3 -> Crystal:Crystal_SMD_Abracon_ABM3-2Pin_5.0x3.2mm
Changed lines of the file:
@@
 F 0 "C2" H 3375 9700 50  0000 L CNN
 F 1 "100nF" H 3375 9500 50  0000 L CNN
-F 2 "Capacitors_SMD:C_0603_HandSoldering" H 3388 9450 30  0001 C CNN
+F 2 "Capacitor_SMD:C_0603_1608Metric_Pad1.05x0.95mm_HandSolder" H 3388 9450 30  0001 C CNN
 F 3 "" H 3350 9600 60  0000 C CNN
 	1    3350 9600
@@
 F 0 "R1" V 2630 1300 50  0000 C CNN
 F 1 "220r" V 2550 1300 50  0000 C CNN
-F 2 "Resistors_SMD:R_0603_HandSoldering" V 2480 1300 30  0001 C CNN
+F 2 "Resistor_SMD:R_0603_1608Metric_Pad1.05x0.95mm_HandSolder" V 2480 1300 30  0001 C CNN
 F 3 "" H 2550 1300 30  0000 C CNN
 	1    2550 1300
@@
 F 0 "C3" H 3675 9700 50  0000 L CNN
 F 1 "100nF" H 3675 9500 50  0000 L CNN
-F 2 "Capacitors_SMD:C_0603_HandSoldering" H 3688 9450 30  0001 C CNN
+F 2 "Capacitor_SMD:C_0603_1608Metric_Pad1.05x0.95mm_HandSolder" H 3688 9450 30  0001 C CNN
 F 3 "" H 3650 9600 60  0000 C CNN
 	1    3650 9600
@@
 F 0 "C5" H 4275 9700 50  0000 L CNN
 F 1 "100nF" H 4275 9500 50  0000 L CNN
-F 2 "Capacitors_SMD:C_0603_HandSoldering" H 4288 9450 30  0001 C CNN
+F 2 "Capacitor_SMD:C_0603_1608Metric_Pad1.05x0.95mm_HandSolder" H 4288 9450 30  0001 C CNN
 F 3 "" H 4250 9600 60  0000 C CNN
 	1    4250 9600
@@
 F 0 "C1" H 9975 8750 50  0000 L CNN
 F 1 "100nF" H 9975 8550 50  0000 L CNN
-F 2 "Capacitors_SMD:C_0603_HandSoldering" H 9988 8500 30  0001 C CNN
+F 2 "Capacitor_SMD:C_0603_1608Metric_Pad1.05x0.95mm_HandSolder" H 9988 8500 30  0001 C CNN
 F 3 "" H 9950 8650 60  0000 C CNN
 	1    9950 8650
@@
 F 0 "C4" H 3975 9700 50  0000 L CNN
 F 1 "100nF" H 3975 9500 50  0000 L CNN
-F 2 "Capacitors_SMD:C_0603_HandSoldering" H 3988 9450 30  0001 C CNN
+F 2 "Capacitor_SMD:C_0603_1608Metric_Pad1.05x0.95mm_HandSolder" H 3988 9450 30  0001 C CNN
 F 3 "" H 3950 9600 60  0000 C CNN
 	1    3950 9600
@@
 F 0 "R2" V 13580 5100 50  0000 C CNN
 F 1 "22r" V 13500 5100 50  0000 C CNN
-F 2 "Resistors_SMD:R_0603_HandSoldering" V 13430 5100 30  0001 C CNN
+F 2 "Resistor_SMD:R_0603_1608Metric_Pad1.05x0.95mm_HandSolder" V 13430 5100 30  0001 C CNN
 F 3 "" H 13500 5100 30  0000 C CNN
 	1    13500 5100
@@
 F 0 "R3" V 13400 5200 50  0000 C CNN
 F 1 "22r" V 13500 5200 50  0000 C CNN
-F 2 "Resistors_SMD:R_0603_HandSoldering" V 13430 5200 30  0001 C CNN
+F 2 "Resistor_SMD:R_0603_1608Metric_Pad1.05x0.95mm_HandSolder" V 13430 5200 30  0001 C CNN
 F 3 "" H 13500 5200 30  0000 C CNN
 	1    13500 5200
@@
 F 0 "DBG1" V 11350 7550 50  0000 L CNN
 F 1 "STRIP_8P" H 11200 8100 50  0000 C BNN
-F 2 "Pin_Headers:Pin_Header_Straight_1x08_Pitch2.54mm" H 11200 8000 60  0001 C CNN
+F 2 "Connector_PinHeader_2.54mm:PinHeader_1x08_P2.54mm_Vertical" H 11200 8000 60  0001 C CNN
 F 3 "" H 11200 8000 60  0000 C CNN
 	1    11050 8000
@@
 F 0 "U3" H 3800 8250 50  0000 C CNN
 F 1 "MCP1700T-3002E/TT" H 3700 8750 50  0000 C CNN
-F 2 "TO_SOT_Packages_SMD:SOT-23" H 3700 8550 50  0001 C CNN
+F 2 "Package_TO_SOT_SMD:SOT-23" H 3700 8550 50  0001 C CNN
 F 3 "" H 3700 8550 50  0000 C CNN
 	1    3700 8450
@@
 F 0 "C10" H 4275 8650 50  0000 L CNN
 F 1 "1uF" H 4275 8450 50  0000 L CNN
-F 2 "Capacitors_SMD:C_0603_HandSoldering" H 4288 8400 50  0001 C CNN
+F 2 "Capacitor_SMD:C_0603_1608Metric_Pad1.05x0.95mm_HandSolder" H 4288 8400 50  0001 C CNN
 F 3 "" H 4250 8550 50  0000 C CNN
 	1    4250 8550
@@
 F 0 "C6" H 3175 8700 50  0000 L CNN
 F 1 "1uF" H 3175 8500 50  0000 L CNN
-F 2 "Capacitors_SMD:C_0603_HandSoldering" H 3188 8450 50  0001 C CNN
+F 2 "Capacitor_SMD:C_0603_1608Metric_Pad1.05x0.95mm_HandSolder" H 3188 8450 50  0001 C CNN
 F 3 "" H 3150 8600 50  0000 C CNN
 	1    3150 8600
@@
 F 0 "P2" H 6650 9150 50  0000 C CNN
 F 1 "CONN_01X04" V 6750 8900 50  0000 C CNN
-F 2 "Pin_Headers:Pin_Header_Straight_1x04_Pitch2.54mm" H 6650 8900 50  0001 C CNN
+F 2 "Connector_PinHeader_2.54mm:PinHeader_1x04_P2.54mm_Vertical" H 6650 8900 50  0001 C CNN
 F 3 "" H 6650 8900 50  0000 C CNN
 	1    6650 8900
@@
 F 0 "EXT1" H 8650 8700 50  0000 C CNN
 F 1 "CONN_01X06" V 8750 8350 50  0000 C CNN
-F 2 "Pin_Headers:Pin_Header_Straight_1x06_Pitch2.54mm" H 8650 8350 50  0001 C CNN
+F 2 "Connector_PinHeader_2.54mm:PinHeader_1x06_P2.54mm_Vertical" H 8650 8350 50  0001 C CNN
 F 3 "" H 8650 8350 50  0000 C CNN
 	1    8650 8350
@@
 F 0 "U1" H 6300 5825 50  0000 L BNN
 F 1 "STM32F042C6Tx" H 12300 5825 50  0000 R BNN
-F 2 "Housings_QFP:LQFP-48_7x7mm_Pitch0.5mm" H 12300 5775 50  0000 R TNN
+F 2 "Package_QFP:LQFP-48_7x7mm_P0.5mm" H 12300 5775 50  0000 R TNN
 F 3 "" H 9300 4100 50  0000 C CNN
 	1    9300 4100
@@
 F 0 "Y1" H 4350 1500 50  0000 C CNN
 F 1 "Crystal" H 4350 1200 50  0000 C CNN
-F 2 "Crystals:ABM3" H 4350 1350 50  0001 C CNN
+F 2 "Crystal:Crystal_SMD_Abracon_ABM3-2Pin_5.0x3.2mm" H 4350 1350 50  0001 C CNN
 F 3 "" H 4350 1350 50  0000 C CNN
 	1    4350 1350
@@
 F 0 "C8" H 4025 1900 50  0000 L CNN
 F 1 "22pF" H 4025 1700 50  0000 L CNN
-F 2 "Capacitors_SMD:C_0603_HandSoldering" H 4038 1650 50  0001 C CNN
+F 2 "Capacitor_SMD:C_0603_1608Metric_Pad1.05x0.95mm_HandSolder" H 4038 1650 50  0001 C CNN
 F 3 "" H 4000 1800 50  0000 C CNN
 	1    4000 1800
@@
 F 0 "C9" H 4825 1900 50  0000 L CNN
 F 1 "22pF" H 4825 1700 50  0000 L CNN
-F 2 "Capacitors_SMD:C_0603_HandSoldering" H 4838 1650 50  0001 C CNN
+F 2 "Capacitor_SMD:C_0603_1608Metric_Pad1.05x0.95mm_HandSolder" H 4838 1650 50  0001 C CNN
 F 3 "" H 4800 1800 50  0000 C CNN
 	1    4800 1800
@@
 F 0 "C11" H 4625 9700 50  0000 L CNN
 F 1 "100nF" H 4625 9500 50  0000 L CNN
-F 2 "Capacitors_SMD:C_0603_HandSoldering" H 4638 9450 50  0001 C CNN
+F 2 "Capacitor_SMD:C_0603_1608Metric_Pad1.05x0.95mm_HandSolder" H 4638 9450 50  0001 C CNN
 F 3 "" H 4600 9600 50  0000 C CNN
 	1    4600 9600
