File: hardware/TCKB.kicad_pcb (KiCad board)
At the start: 2 copper layers, 285 x 94.6 mm, 242 parts, among them J1 USB-MB-H, P2 CONN_01X04, SW10 k_7, SW11 k_8, SW12 k_9, SW13 k_0, SW14 k_MINUS, SW15 k_EQUAL, SW16 k_BSPACE, SW17 k_TAB, SW18 k_Q, SW19 k_W, SW20 k_E, SW21 k_R, SW22 k_T, SW23 k_Y, SW24 k_U, SW25 k_I, SW26 k_O, SW27 k_P, SW28 k_LBRACKET, SW29 k__RBRACKET, SW3 k_ESC, SW30 k_BSLASH_ANSI, SW31 k_CAPSLOCK, SW32 k_A, SW33 k_S, SW34 k_D, SW35 k_F, SW36 k_G, SW37 k_H, SW38 k_J, SW39 k_K, SW4 k_1, SW40 k_L, SW41 k_SEMICOLON, SW42 k_QUOTE, SW43 k_BSLASH_ISO, SW44 k_ENTER_ISO, SW45 k_ENTER_ANSI, SW46 k_LSHIFT_ISO, SW47 k_NU_BSLASH_ISO, SW48 k_Z, SW49 k_X, SW5 k_2, SW50 k_C, SW51 k_V, SW52 k_B, SW53 k_N, SW54 k_M, SW55 k_COMMA, SW56 k_DOT, SW57 k_SLASH, SW58 k_RSHIFT, SW59 k_LSHIFT_ANSI, SW6 k_3, SW60 k_LCTRL, SW61 k_LGUI, SW62 k_LALT, SW63 k_SPACE, SW64 k_RALT, SW65 k_RGUI, SW66 k_RMENU, SW67 k_RCTRL, SW7 k_4, SW8 k_5, SW9 k_6, U1 STM32F042C6Tx, U3 MCP1700T-3002E/TT, U5 IS31FL3733, Y1 Crystal

Commit message: Update TCKB.kicad_pcb
Parts:
- C1, C10, C11, C19, C2, C20, C21, C22, C23, C24, C25, C3, C4, C5, C6, C8, C9: footprint Capacitors_SMD:C_0603_HandSoldering -> Capacitor_SMD:C_0603_1608Metric_Pad1.05x0.95mm_HandSolder
- C7: footprint Capacitors_SMD:C_1206_HandSoldering -> Capacitor_SMD:C_1206_3216Metric_Pad1.42x1.75mm_HandSolder
- D10, D11, D12, D13, D14, D15, D16, D17, D18, D19, D20, D21, D22, D23, D24, D25, D26, D27, D28, D29, D3, D30, D31, D32, D33, D34, D35, D36, D37, D38, D39, D4, D40, D41, D42, D43, D44, D45, D46, D47, D48, D49, D5, D50, D51, D52, D53, D54, D55, D56, D57, D58, D59, D6, D60, D61, D62, D63, D64, D65, D7, D8, D9: footprint TCKB:MiniMELF_2mm -> Diode_SMD:D_MiniMELF
- DBG1: footprint Pin_Headers:Pin_Header_Straight_1x08_Pitch2.54mm -> Connector_PinHeader_2.54mm:PinHeader_1x08_P2.54mm_Vertical
- EXT1: footprint Pin_Headers:Pin_Header_Straight_1x06_Pitch2.54mm -> Connector_PinHeader_2.54mm:PinHeader_1x06_P2.54mm_Vertical
- J1: footprint SparkFun-Connectors:USB-MB-H -> TCKB:USB-MB-H
- P2: footprint Pin_Headers:Pin_Header_Straight_1x04_Pitch2.54mm -> Connector_PinHeader_2.54mm:PinHeader_1x04_P2.54mm_Vertical
- R1, R2, R3, R4, R5, R6, R7, R8, R9: footprint Resistors_SMD:R_0603_HandSoldering -> Resistor_SMD:R_0603_1608Metric_Pad1.05x0.95mm_HandSolder
- U1: footprint Housings_QFP:LQFP-48_7x7mm_Pitch0.5mm -> Package_QFP:LQFP-48_7x7mm_P0.5mm
- U3: footprint TO_SOT_Packages_SMD:SOT-23 -> Package_TO_SOT_SMD:SOT-23
- U5: footprint Housings_DFN_QFN:UQFN-48-1EP_6x6mm_Pitch0.4mm -> Package_DFN_QFN:UQFN-48-1EP_6x6mm_P0.4mm_EP4.45x4.45mm
- Y1: footprint Crystals:ABM3 -> Crystal:Crystal_SMD_Abracon_ABM3-2Pin_5.0x3.2mm
