File: hardware/Matrix.sch (KiCad schematic (older format))
At the start: 134 parts, among them SW10 k_7, SW11 k_8, SW12 k_9, SW13 k_0, SW14 k_MINUS, SW15 k_EQUAL, SW16 k_BSPACE, SW17 k_TAB, SW18 k_Q, SW19 k_W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

Commit message: Update Matrix.sch
Parts:
- D10, D11, D12, D13, D14, D15, D16, D17, D18, D19, D20, D21, D22, D23, D24, D25, D26, D27, D28, D29, D3, D30, D31, D32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: footprint TCKB:MiniMELF_2mm -> Diode_SMD:D_MiniMELF
